File: hardware/avr-batt-timer/avr-batt-timer.kicad_pcb (KiCad board)
At the start: 2 copper layers, 25.5 x 56.9 mm, 13 parts, among them J1 XT60PW-M, J2 XT60PW-F, J3 Conn_01x05_Pin, U1 ATtiny5-TS, U2 L78L05_SOT89

Commit message: +1
Parts:
- moved D1 31.5 mm to (149.1, 72.4)
- moved J3 20.6 mm to (149.1, 114.6), turned to 180 degrees
- moved J1 2.71 mm to (140.3, 112.3)
- moved J2 2.10 mm to (140.5, 70.7)
- moved R1 0.33 mm to (134.3, 90.7), turned to 0 degrees
Connections:
- R1 pad 1: VCC -> VDD
Routing:
- net LOAD: track 0.00 -> 71.4 mm
- net VDD: track 0.00 -> 57.4 mm, vias 0 -> 1
- net +5V: track 0.00 -> 39.6 mm
- net TPIDATA: track 0.00 -> 25.6 mm, vias 0 -> 1
- net RESET: track 0.00 -> 21.5 mm, vias 0 -> 1
- net Net-(D1-A): track 0.00 -> 19.6 mm, vias 0 -> 1
- net TPICLK: track 0.00 -> 16.5 mm
- net Net-(MOSFET1-G): track 0.00 -> 8.93 mm
- net VSENSE: track 0.00 -> 8.38 mm
- added copper zone on B.Cu, net GND
- added copper zone on F.Cu, net VDD
Other:
- outline, holes or cut-outs redrawn

Commit message: +1
Parts:
- D2: value D -> D 15A
- MOSFET1: value IRFZ44N_127 -> IRFZ44N; footprint Package_TO_SOT_THT:TO-220-2_Horizontal_TabDown -> Package_TO_SOT_THT:TO-220-3_Horizontal_TabDown
- R3: value ~ 250R -> ~250R
- R4: value ~ 10K -> ~10K
- R5: value ~ 700R -> ~700R
- U1: value ATtiny5-TS -> ATtiny5
- moved D2 25.3 mm to (153.2, 90.4), turned to 90 degrees
- moved MOSFET1 20.1 mm to (153.1, 78.9)
- moved U2 19.5 mm to (141.6, 102.3)
- moved J1 15.5 mm to (145.3, 97.7)
- moved R4 13.0 mm to (136.3, 82.5), turned to -90 degrees
- moved J3 9.66 mm to (153.7, 106.1)
- moved U1 9.16 mm to (143.5, 88.4), turned to 90 degrees
- moved D1 7.11 mm to (153.5, 66.8)
- moved J2 7.00 mm to (146.0, 66.3)
- moved R5 6.57 mm to (147.2, 82.9), turned to 0 degrees
- moved R3 5.99 mm to (148.4, 91.7), turned to -90 degrees
- moved R1 5.33 mm to (139.1, 92.9)
- moved R2 4.63 mm to (143.3, 92.9)
Routing:
- net LOAD: track 71.4 -> 0.15 mm
- net Net-(MOSFET1-G): track 8.93 -> 27.8 mm
- net TPIDATA: track 25.6 -> 16.4 mm
- net Net-(D1-A): track 19.6 -> 15.2 mm, vias 1 -> 0
- net VDD: track 57.4 -> 53.1 mm, vias 1 -> 3
- net GND: track 0.00 -> 3.46 mm
- net VSENSE: track 8.38 -> 5.09 mm
- net +5V: track 39.6 -> 37.3 mm, vias 0 -> 2
- net TPICLK: track 16.5 -> 18.6 mm, vias 0 -> 1
- net RESET: track 21.5 -> 21.8 mm, vias 1 -> 0
- added copper zone on F.Cu, net LOAD
- removed copper zone on F.Cu, net VDD
Other:
- board size 25.5 x 56.9 mm -> 24.1 x 49.9 mm
- board text added: "+5V"
- board text added: "GND"
- board text added: "RST"
- board text added: "TCLK"
- board text added: "TDAT"

Commit message: +1
Routing:
- net VDD: track 53.1 -> 44.7 mm
Changed lines of the file:
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@@
 			(drillshape 0)
 			(scaleselection 1)
-			(outputdirectory "")
+			(outputdirectory "../../../../Downloads/avr-batt-timer/")
 		)
 	)
@@
 			(pinfunction "1")
 			(pintype "passive")
+			(thermal_bridge_width 3)
+			(thermal_bridge_angle 45)
 		)
 		(pad "2" thru_hole circle
@@
 			(pinfunction "1")
 			(pintype "passive")
-			(thermal_bridge_width 1.25)
+			(thermal_bridge_width 2)
 		)
 		(pad "2" thru_hole circle
@@
 			(pinfunction "K")
 			(pintype "passive")
-			(thermal_bridge_width 1)
+			(thermal_bridge_width 1.5)
 		)
 		(pad "2" thru_hole circle
@@
 			(pinfunction "A")
 			(pintype "passive")
-			(thermal_bridge_width 1)
+			(thermal_bridge_width 1.5)
 		)
 		(model "${KICAD8_3DMODEL_DIR}/Package_TO_SOT_THT.3dshapes/TO-220-2_Horizontal_TabDown.wrl"
@@
 			(pinfunction "D")
 			(pintype "unspecified")
-			(thermal_bridge_width 1.2)
+			(thermal_bridge_width 1.7)
 			(thermal_bridge_angle 45)
 		)
@@
 			(pinfunction "S")
 			(pintype "unspecified")
-			(thermal_bridge_width 1)
+			(thermal_bridge_width 1.7)
 			(thermal_bridge_angle 45)
 		)
@@
 		(tags "resistor handsolder")
 		(property "Reference" "R5"
-			(at 0 1.65 360)
+			(at 0 1.65 0)
 			(layer "B.SilkS")
 			(effects
@@
 		)
 		(fp_text user "${REFERENCE}"
-			(at 0 0 360)
+			(at 0 0 0)
 			(layer "B.Fab")
 			(effects
@@
 		)
 	)
+	(gr_poly
+		(pts
+			(xy 144.5768 69.342) (xy 146.9644 74.8792) (xy 147.828 79.6544) (xy 147.9296 85.09) (xy 147.1676 86.6394)
+			(xy 147.2184 87.6808) (xy 146.7358 88.9762) (xy 145.6182 92.3544)
+		)
+		(stroke
+			(width 0.2)
+			(type solid)
+		)
+		(fill solid)
+		(layer "F.Cu")
+		(net 4)
+	)
+	(gr_poly
+		(pts
+			(xy 139.2174 100.8888) (xy 142.1892 99.2124) (xy 143.1036 95.7072) (xy 145.6182 92.3544) (xy 138.6586 91.7956)
+			(xy 135.8392 94.6912) (xy 135.577643 97.663) (xy 135.8392 99.568) (xy 137.3886 100.457) (xy 139.2682 100.8888)
+		)
+		(stroke
+			(width 0.2)
+			(type solid)
+		)
+		(fill solid)
+		(layer "F.Cu")
+		(net 4)
+	)
+	(gr_poly
+		(pts
+			(xy 139.2174 88.0872) (xy 140.2334 89.7636) (xy 138.6586 91.7956) (xy 135.8392 94.6912)
+		)
+		(stroke
+			(width 0.2)
+			(type solid)
+		)
+		(fill solid)
+		(layer "F.Cu")
+		(net 4)
+	)
+	(gr_poly
+		(pts
+			(xy 139.0142 79.2734) (xy 138.8618 75.9206) (xy 138.0236 74.168) (xy 135.9916 72.1868) (xy 141.097 72.7202)
+			(xy 140.3096 79.5782)
+		)
+		(stroke
+			(width 0.2)
+			(type solid)
+		)
+		(fill solid)
+		(layer "F.Cu")
+		(net 4)
+	)
 	(gr_circle
 		(center 138.0998 97.663)
@@
 		(net 4)
 	)
+	(gr_poly
+		(pts
+			(xy 139.1412 77.0128) (xy 136.398 79.2988) (xy 136.2456 84.7344) (xy 138.5824 86.4616) (xy 139.3444 87.2236)
+		)
+		(stroke
+			(width 0.2)
+			(type solid)
+		)
+		(fill solid)
+		(layer "F.Cu")
+		(net 4)
+	)
+	(gr_poly
+		(pts
+			(xy 141.1986 64.008) (xy 144.5768 69.342) (xy 145.7706 72.9488) (xy 138.8618 71.0184) (xy 141.1986 63.9318)
+		)
+		(stroke
+			(width 0.2)
+			(type solid)
+		)
+		(fill solid)
+		(layer "F.Cu")
+		(net 4)
+	)
 	(gr_line
 		(start 154.337 108.5596)
@@
 	)
 	(segment
-		(start 138.132 94.1256)
-		(end 138.132 97.6504)
-		(width 5)
+		(start 142.4432 90.932)
+		(end 142.4432 73.787)
+		(width 7)
 		(layer "F.Cu")
 		(net 4)
 	)
 	(segment
-		(start 138.7856 69.342)
-		(end 142.367 72.9234)
-		(width 5)
-		(layer "F.Cu")
-		(net 4)
-	)
-	(segment
-		(start 142.367 72.9234)
-		(end 142.367 79.3242)
-		(width 5)
+		(start 142.4432 73.787)
+		(end 138.7924 70.1362)
+		(width 7)
 		(layer "F.Cu")
 		(net 4)
@@
 	)
 	(segment
-		(start 142.367 89.8906)
-		(end 138.132 94.1256)
-		(width 5)
-		(layer "F.Cu")
-		(net 4)
-	)
-	(segment
-		(start 138.7924 69.3352)
+		(start 138.7924 70.1362)
 		(end 138.7924 66.3146)
-		(width 5)
-		(layer "F.Cu")
-		(net 4)
-	)
-	(segment
-		(start 142.367 79.3242)
-		(end 142.367 89.8906)
-		(width 5)
+		(width 7)
 		(layer "F.Cu")
 		(net 4)
@@
 	)
 	(segment
-		(start 138.7856 69.342)
-		(end 138.7924 69.3352)
-		(width 5)
-		(layer "F.Cu")
-		(net 4)
-	)
-	(segment
 		(start 138.43 104.2416)
 		(end 138.43 97.9484)
@@
 	)
 	(segment
-		(start 148.8694 100.33)
-		(end 144.9324 104.267)
+		(start 147.8026 87.122)
+		(end 148.8694 88.1888)
 		(width 0.2)
 		(layer "F.Cu")
@@
 	)
 	(segment
-		(start 147.32 86.9442)
-		(end 148.8694 88.4936)
+		(start 148.8694 88.1888)
+		(end 148.8694 100.33)
 		(width 0.2)
 		(layer "F.Cu")
@@
 	)
 	(segment
-		(start 148.8694 88.4936)
-		(end 148.8694 100.33)
+		(start 144.9324 104.267)
+		(end 146.7358 106.0704)
 		(width 0.2)
 		(layer "F.Cu")
@@
 	)
 	(segment
-		(start 144.9324 104.267)
-		(end 146.7358 106.0704)
+		(start 148.8694 100.33)
+		(end 144.9324 104.267)
 		(width 0.2)
 		(layer "F.Cu")
@@
 	)
 	(via
-		(at 147.32 86.9442)
+		(at 147.8026 87.122)
 		(size 0.6)
 		(drill 0.3)
@@
 	)
 	(segment
-		(start 143.0542 104.2358)
-		(end 144.9012 104.2358)
+		(start 147.8026 87.122)
+		(end 145.9484 85.2678)
 		(width 0.2)
 		(layer "B.Cu")
@@
 	)
 	(segment
-		(start 143.4592 85.5218)
-		(end 143.7132 85.2678)
+		(start 143.0542 104.2358)
+		(end 144.9012 104.2358)
 		(width 0.2)
 		(layer "B.Cu")
@@
 	)
 	(segment
-		(start 145.6436 85.2678)
-		(end 147.32 86.9442)
+		(start 143.7132 85.2678)
+		(end 143.4592 85.5218)
 		(width 0.2)
 		(layer "B.Cu")
@@
 	)
 	(segment
-		(start 143.4592 87.0928)
-		(end 143.4592 85.5218)
+		(start 143.4592 85.5218)
+		(end 143.4592 87.0928)
 		(width 0.2)
 		(layer "B.Cu")
@@
 	)
 	(segment
-		(start 143.7132 85.2678)
-		(end 145.6436 85.2678)
+		(start 145.9484 85.2678)
+		(end 143.7132 85.2678)
 		(width 0.2)
 		(layer "B.Cu")
